Commit message: Add files via upload

File: packages/erp42_vehicle/erp42_vehicle_description/urdf/erp42_vehicle.urdf.xacro (robot description, xacro)
@@ -152,4 +152,13 @@
    <link name="imu_link">
    </link>
+    <!-- GPS link -->
+  <joint name="gps_joint" type="fixed">
+    <axis xyz="0 0 1" />
+    <origin xyz="0 0 0.2" rpy="0 0 0"/>
+    <parent link="base_link"/>
+    <child link="gps_link"/>
+  </joint>
+  <link name="gps_link">
+  </link>
      <!-- Camera -->
   <joint name="camera_joint" type="fixed">
@@ -242,3 +251,16 @@
     </plugin>
   </gazebo>
+  <gazebo>
+    <plugin name="gps_plugin" filename="libhector_gazebo_ros_gps.so">
+      <alwaysOn>true</alwaysOn>
+      <bodyName>gps_link</bodyName>
+      <topicName>fix</topicName>
+      <velocitytopicName>fixvelocity</velocitytopicName>
+      <drift>0.0 0.0 0.0</drift>
+      <gaussianNoise>0.1 0.1 0.1</gaussianNoise>
+      <velocitydrift>0 0 0</velocitydrift>
+      <velocitygaussianNoise>0.1 0.1 0.1</velocitygaussianNoise>
+      <updateRate>10.0</updateRate>
+    </plugin>
+  </gazebo>
 </robot>

Commit message: Add files via upload

File: packages/erp42_vehicle/erp42_vehicle_description/urdf/erp42_vehicle.urdf.xacro (robot description, xacro)
@@ -146,18 +146,44 @@
    <joint name="imu_joint" type="fixed">
     <axis xyz="0 0 1" />
-    <origin xyz="0 0 0.02" rpy="0 0 0"/>
+    <origin xyz="0.2 0 0.14" rpy="0 0 0"/>
     <parent link="base_link"/>
     <child link="imu_link"/>
    </joint>
    <link name="imu_link">
+    <visual>
+      <origin xyz="0 0 0" rpy="0 0 0"/>
+      <geometry>
+        <box size="0.04 0.04 0.02"/>
+      </geometry>
+      <material name="blue" />
+    </visual>
+    <collision>
+      <origin xyz="0 0 0" rpy="0 0 0"/>
+      <geometry>
+        <box size="0.04 0.04 0.02"/>
+      </geometry>
+    </collision>
    </link>
     <!-- GPS link -->
   <joint name="gps_joint" type="fixed">
     <axis xyz="0 0 1" />
-    <origin xyz="0 0 0.2" rpy="0 0 0"/>
+    <origin xyz="0.2 0 0.25" rpy="0 0 0"/>
     <parent link="base_link"/>
     <child link="gps_link"/>
   </joint>
   <link name="gps_link">
+    <visual>
+      <origin xyz="0 0 0" rpy="0 0 0"/>
+      <geometry>
+        <box size="0.04 0.04 0.02"/>
+      </geometry>
+      <material name="blue" />
+    </visual>
+    <collision>
+      <origin xyz="0 0 0" rpy="0 0 0"/>
+      <geometry>
+        <box size="0.04 0.04 0.02"/>
+      </geometry>
+    </collision>
   </link>
      <!-- Camera -->
